Commit message: added ros2_control interface and changed pkg name

File: my_robot_bringup/urdf/robo_desc.xacro (robot description, xacro)
@@ -24,19 +24,19 @@
       <geometry>
         <mesh
-          filename="package://my_robot_description/meshes/base_link.STL" />
-      </geometry>
-      <material
-        name="">
-        <color
-          rgba="0.79216 0.81961 0.93333 1" />
-      </material>
-    </visual>
-    <collision>
-      <origin
-        xyz="0 0 0"
-        rpy="0 0 0" />
-      <geometry>
-        <mesh
-          filename="package://my_robot_description/meshes/base_link.STL" />
+          filename="package://my_robot_bringup/meshes/base_link.STL" />
+      </geometry>
+      <material
+        name="">
+        <color
+          rgba="0.79216 0.81961 0.93333 1" />
+      </material>
+    </visual>
+    <collision>
+      <origin
+        xyz="0 0 0"
+        rpy="0 0 0" />
+      <geometry>
+        <mesh
+          filename="package://my_robot_bringup/meshes/base_link.STL" />
       </geometry>
     </collision>
@@ -64,19 +64,19 @@
       <geometry>
         <mesh
-          filename="package://my_robot_description/meshes/fl_shoulder.STL" />
-      </geometry>
-      <material
-        name="">
-        <color
-          rgba="0.79216 0.81961 0.93333 1" />
-      </material>
-    </visual>
-    <collision>
-      <origin
-        xyz="0 0 0"
-        rpy="0 0 0" />
-      <geometry>
-        <mesh
-          filename="package://my_robot_description/meshes/fl_shoulder.STL" />
+          filename="package://my_robot_bringup/meshes/fl_shoulder.STL" />
+      </geometry>
+      <material
+        name="">
+        <color
+          rgba="0.79216 0.81961 0.93333 1" />
+      </material>
+    </visual>
+    <collision>
+      <origin
+        xyz="0 0 0"
+        rpy="0 0 0" />
+      <geometry>
+        <mesh
+          filename="package://my_robot_bringup/meshes/fl_shoulder.STL" />
       </geometry>
     </collision>
@@ -122,5 +122,5 @@
       <geometry>
         <mesh
-          filename="package://my_robot_description/meshes/fl_femur.STL" />
+          filename="package://my_robot_bringup/meshes/fl_femur.STL" />
       </geometry>
       <material
@@ -136,5 +136,5 @@
       <geometry>
         <mesh
-          filename="package://my_robot_description/meshes/fl_femur.STL" />
+          filename="package://my_robot_bringup/meshes/fl_femur.STL" />
       </geometry>
     </collision>
@@ -180,5 +180,5 @@
       <geometry>
         <mesh
-          filename="package://my_robot_description/meshes/fl_tibia.STL" />
+          filename="package://my_robot_bringup/meshes/fl_tibia.STL" />
       </geometry>
       <material
@@ -194,5 +194,5 @@
       <geometry>
         <mesh
-          filename="package://my_robot_description/meshes/fl_tibia.STL" />
+          filename="package://my_robot_bringup/meshes/fl_tibia.STL" />
       </geometry>
     </collision>
@@ -238,19 +238,19 @@
       <geometry>
         <mesh
-          filename="package://my_robot_description/meshes/fr_shoulder.STL" />
-      </geometry>
-      <material
-        name="">
-        <color
-          rgba="0.79216 0.81961 0.93333 1" />
-      </material>
-    </visual>
-    <collision>
-      <origin
-        xyz="0 0 0"
-        rpy="0 0 0" />
-      <geometry>
-        <mesh
-          filename="package://my_robot_description/meshes/fr_shoulder.STL" />
+          filename="package://my_robot_bringup/meshes/fr_shoulder.STL" />
+      </geometry>
+      <material
+        name="">
+        <color
+          rgba="0.79216 0.81961 0.93333 1" />
+      </material>
+    </visual>
+    <collision>
+      <origin
+        xyz="0 0 0"
+        rpy="0 0 0" />
+      <geometry>
+        <mesh
+          filename="package://my_robot_bringup/meshes/fr_shoulder.STL" />
       </geometry>
     </collision>
@@ -296,5 +296,5 @@
       <geometry>
         <mesh
-          filename="package://my_robot_description/meshes/fr_femur.STL" />
+          filename="package://my_robot_bringup/meshes/fr_femur.STL" />
       </geometry>
       <material
@@ -310,5 +310,5 @@
       <geometry>
         <mesh
-          filename="package://my_robot_description/meshes/fr_femur.STL" />
+          filename="package://my_robot_bringup/meshes/fr_femur.STL" />
       </geometry>
     </collision>
@@ -354,5 +354,5 @@
       <geometry>
         <mesh
-          filename="package://my_robot_description/meshes/fr_tibia.STL" />
+          filename="package://my_robot_bringup/meshes/fr_tibia.STL" />
       </geometry>
       <material
@@ -368,5 +368,5 @@
       <geometry>
         <mesh
-          filename="package://my_robot_description/meshes/fr_tibia.STL" />
+          filename="package://my_robot_bringup/meshes/fr_tibia.STL" />
       </geometry>
     </collision>
@@ -412,19 +412,19 @@
       <geometry>
         <mesh
-          filename="package://my_robot_description/meshes/bl_shoulder.STL" />
-      </geometry>
-      <material
-        name="">
-        <color
-          rgba="0.79216 0.81961 0.93333 1" />
-      </material>
-    </visual>
-    <collision>
-      <origin
-        xyz="0 0 0"
-        rpy="0 0 0" />
-      <geometry>
-        <mesh
-          filename="package://my_robot_description/meshes/bl_shoulder.STL" />
+          filename="package://my_robot_bringup/meshes/bl_shoulder.STL" />
+      </geometry>
+      <material
+        name="">
+        <color
+          rgba="0.79216 0.81961 0.93333 1" />
+      </material>
+    </visual>
+    <collision>
+      <origin
+        xyz="0 0 0"
+        rpy="0 0 0" />
+      <geometry>
+        <mesh
+          filename="package://my_robot_bringup/meshes/bl_shoulder.STL" />
       </geometry>
     </collision>
@@ -470,19 +470,19 @@
       <geometry>
         <mesh
-          filename="package://my_robot_description/meshes/bl_femur.STL" />
-      </geometry>
-      <material
-        name="">
-        <color
-          rgba="0.79216 0.81961 0.93333 1" />
-      </material>
-    </visual>
-    <collision>
-      <origin
-        xyz="0 0 0"
-        rpy="0 0 0" />
-      <geometry>
-        <mesh
-          filename="package://my_robot_description/meshes/bl_femur.STL" />
+          filename="package://my_robot_bringup/meshes/bl_femur.STL" />
+      </geometry>
+      <material
+        name="">
+        <color
+          rgba="0.79216 0.81961 0.93333 1" />
+      </material>
+    </visual>
+    <collision>
+      <origin
+        xyz="0 0 0"
+        rpy="0 0 0" />
+      <geometry>
+        <mesh
+          filename="package://my_robot_bringup/meshes/bl_femur.STL" />
       </geometry>
     </collision>
@@ -528,19 +528,19 @@
       <geometry>
         <mesh
-          filename="package://my_robot_description/meshes/bl_tibia.STL" />
-      </geometry>
-      <material
-        name="">
-        <color
-          rgba="0.79216 0.81961 0.93333 1" />
-      </material>
-    </visual>
-    <collision>
-      <origin
-        xyz="0 0 0"
-        rpy="0 0 0" />
-      <geometry>
-        <mesh
-          filename="package://my_robot_description/meshes/bl_tibia.STL" />
+          filename="package://my_robot_bringup/meshes/bl_tibia.STL" />
+      </geometry>
+      <material
+        name="">
+        <color
+          rgba="0.79216 0.81961 0.93333 1" />
+      </material>
+    </visual>
+    <collision>
+      <origin
+        xyz="0 0 0"
+        rpy="0 0 0" />
+      <geometry>
+        <mesh
+          filename="package://my_robot_bringup/meshes/bl_tibia.STL" />
       </geometry>
     </collision>
@@ -586,19 +586,19 @@
       <geometry>
         <mesh
-          filename="package://my_robot_description/meshes/br_shoulder.STL" />
-      </geometry>
-      <material
-        name="">
-        <color
-          rgba="0.79216 0.81961 0.93333 1" />
-      </material>
-    </visual>
-    <collision>
-      <origin
-        xyz="0 0 0"
-        rpy="0 0 0" />
-      <geometry>
-        <mesh
-          filename="package://my_robot_description/meshes/br_shoulder.STL" />
+          filename="package://my_robot_bringup/meshes/br_shoulder.STL" />
+      </geometry>
+      <material
+        name="">
+        <color
+          rgba="0.79216 0.81961 0.93333 1" />
+      </material>
+    </visual>
+    <collision>
+      <origin
+        xyz="0 0 0"
+        rpy="0 0 0" />
+      <geometry>
+        <mesh
+          filename="package://my_robot_bringup/meshes/br_shoulder.STL" />
       </geometry>
     </collision>
@@ -644,19 +644,19 @@
       <geometry>
         <mesh
-          filename="package://my_robot_description/meshes/br_femur.STL" />
-      </geometry>
-      <material
-        name="">
-        <color
-          rgba="0.79216 0.81961 0.93333 1" />
-      </material>
-    </visual>
-    <collision>
-      <origin
-        xyz="0 0 0"
-        rpy="0 0 0" />
-      <geometry>
-        <mesh
-          filename="package://my_robot_description/meshes/br_femur.STL" />
+          filename="package://my_robot_bringup/meshes/br_femur.STL" />
+      </geometry>
+      <material
+        name="">
+        <color
+          rgba="0.79216 0.81961 0.93333 1" />
+      </material>
+    </visual>
+    <collision>
+      <origin
+        xyz="0 0 0"
+        rpy="0 0 0" />
+      <geometry>
+        <mesh
+          filename="package://my_robot_bringup/meshes/br_femur.STL" />
       </geometry>
     </collision>
@@ -702,19 +702,19 @@
       <geometry>
         <mesh
-          filename="package://my_robot_description/meshes/br_tibia.STL" />
-      </geometry>
-      <material
-        name="">
-        <color
-          rgba="0.79216 0.81961 0.93333 1" />
-      </material>
-    </visual>
-    <collision>
-      <origin
-        xyz="0 0 0"
-        rpy="0 0 0" />
-      <geometry>
-        <mesh
-          filename="package://my_robot_description/meshes/br_tibia.STL" />
+          filename="package://my_robot_bringup/meshes/br_tibia.STL" />
+      </geometry>
+      <material
+        name="">
+        <color
+          rgba="0.79216 0.81961 0.93333 1" />
+      </material>
+    </visual>
+    <collision>
+      <origin
+        xyz="0 0 0"
+        rpy="0 0 0" />
+      <geometry>
+        <mesh
+          filename="package://my_robot_bringup/meshes/br_tibia.STL" />
       </geometry>
     </collision>
@@ -731,5 +731,5 @@
       link="br_tibia" />
     <axis
-      xyz="0 0 1" />
+      xyz="0 0 -1" />
     <limit
       lower="-1.57"
